File: Layout and PCB/68030-TK-V09c.sch (EAGLE design)
At the start: 65 parts, among them IC10 74HCT245DW, IC11 74HCT245DW, IC4 74HCT245DW, IC5 74HCT245DW, IC6 74HCT245DW, IC8 74HCT245DW, IC9 74HCT245DW, X1 FABC96R

Commit message: minor clean up
Parts:
- added R17: 4,7k, rcl:R-EU_R0603
Connections:
- removed net RW_OUT: IC7.IO23, IC9A.A1
- new net AMIGA_ADR_ENABLE: IC4A.G, IC7.IO29, IC8A.G, IC9A.G
- net A6: now also IC7.IO23; no longer IC7.IO33
- net AS_00: now also IC7.IO33; no longer IC7.IO29
- net AVEC: now also R17.2
- net GND: no longer IC4A.G, IC8A.G, IC9A.G
- net R/W: now also IC9A.A1
- net VCC: now also R17.1
Changed lines of the file:
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@@
 <part name="R14" library="rcl" deviceset="R-EU_" device="R0603"/>
 <part name="R16" library="rcl" deviceset="R-EU_" device="R0603"/>
+<part name="R17" library="rcl" deviceset="R-EU_" device="R0603" value="4,7k"/>
 </parts>
 <sheets>
@@
 <instance part="R8" gate="G$1" x="-2.54" y="121.92"/>
 <instance part="R9" gate="G$1" x="-2.54" y="116.84"/>
+<instance part="R17" gate="G$1" x="-2.54" y="93.98"/>
 </instances>
 <busses>
@@
 <label x="91.44" y="124.46" size="1.27" layer="95" rot="R180" xref="yes"/>
 </segment>
+<segment>
+<pinref part="R17" gate="G$1" pin="2"/>
+<wire x1="2.54" y1="93.98" x2="10.16" y2="93.98" width="0.1524" layer="91"/>
+<label x="10.16" y="93.98" size="1.778" layer="95"/>
+</segment>
 </net>
 <net name="CIIN" class="0">
@@
 <wire x1="-7.62" y1="116.84" x2="-20.32" y2="116.84" width="0.1524" layer="91"/>
 <pinref part="R2" gate="G$1" pin="2"/>
-<wire x1="-20.32" y1="91.44" x2="-20.32" y2="101.6" width="0.1524" layer="91"/>
+<wire x1="-20.32" y1="91.44" x2="-20.32" y2="93.98" width="0.1524" layer="91"/>
 <junction x="-20.32" y="101.6"/>
+<pinref part="R17" gate="G$1" pin="1"/>
+<wire x1="-20.32" y1="93.98" x2="-20.32" y2="101.6" width="0.1524" layer="91"/>
+<wire x1="-7.62" y1="93.98" x2="-20.32" y2="93.98" width="0.1524" layer="91"/>
+<junction x="-20.32" y="93.98"/>
 </segment>
 <segment>
@@
 </segment>
 </net>
-<net name="AS_00" class="0">
-<segment>
-<pinref part="IC7" gate="G$1" pin="IO29"/>
-<wire x1="101.6" y1="25.4" x2="101.6" y2="30.48" width="0.1524" layer="91"/>
-<label x="101.6" y="25.4" size="1.27" layer="95" rot="R270"/>
-</segment>
-</net>
 <net name="CS_FPU" class="0">
 <segment>
@@
 <net name="AVEC" class="0">
 <segment>
-<pinref part="IC7" gate="G$1" pin="IO1"/>
-<wire x1="104.14" y1="116.84" x2="104.14" y2="121.92" width="0.1524" layer="91"/>
-<label x="104.14" y="121.92" size="1.27" layer="95" rot="R90"/>
-</segment>
-<segment>
 <label x="238.76" y="76.2" size="1.27" layer="95" xref="yes"/>
 <pinref part="X1" gate="-A13" pin="B"/>
 <wire x1="236.22" y1="76.2" x2="238.76" y2="76.2" width="0.1524" layer="91"/>
 </segment>
+<segment>
+<pinref part="IC7" gate="G$1" pin="IO1"/>
+<wire x1="104.14" y1="116.84" x2="104.14" y2="121.92" width="0.1524" layer="91"/>
+<label x="104.14" y="121.92" size="1.27" layer="95" rot="R90"/>
+</segment>
 </net>
 <net name="BG_30" class="0">
@@
 </segment>
 <segment>
-<pinref part="IC7" gate="G$1" pin="IO33"/>
-<wire x1="124.46" y1="30.48" x2="124.46" y2="27.94" width="0.1524" layer="91"/>
-<label x="124.46" y="27.94" size="1.27" layer="95" rot="R270"/>
+<pinref part="IC7" gate="G$1" pin="IO23"/>
+<wire x1="71.12" y1="50.8" x2="66.04" y2="50.8" width="0.1524" layer="91"/>
+<label x="66.04" y="50.8" size="1.27" layer="95" rot="R180"/>
 </segment>
 </net>
@@
 </segment>
 </net>
-<net name="RW_OUT" class="0">
+<net name="AMIGA_ADR_ENABLE" class="0">
 <segment>
-<pinref part="IC7" gate="G$1" pin="IO23"/>
-<wire x1="71.12" y1="50.8" x2="66.04" y2="50.8" width="0.1524" layer="91"/>
-<label x="66.04" y="50.8" size="1.27" layer="95" rot="R180"/>
+<pinref part="IC7" gate="G$1" pin="IO29"/>
+<wire x1="101.6" y1="25.4" x2="101.6" y2="30.48" width="0.1524" layer="91"/>
+<label x="101.6" y="25.4" size="1.27" layer="95" rot="R270"/>
+</segment>
+</net>
+<net name="AS_00" class="0">
+<segment>
+<pinref part="IC7" gate="G$1" pin="IO33"/>
+<wire x1="124.46" y1="30.48" x2="124.46" y2="27.94" width="0.1524" layer="91"/>
+<label x="124.46" y="27.94" size="1.27" layer="95" rot="R270"/>
 </segment>
 </net>
@@
 <junction x="111.76" y="12.7"/>
 </segment>
-<segment>
-<pinref part="IC4" gate="A" pin="G"/>
-<wire x1="40.64" y1="139.7" x2="45.72" y2="139.7" width="0.1524" layer="91"/>
-<label x="45.72" y="139.7" size="1.27" layer="95"/>
-</segment>
-<segment>
-<pinref part="IC8" gate="A" pin="G"/>
-<wire x1="40.64" y1="99.06" x2="45.72" y2="99.06" width="0.1524" layer="91"/>
-<label x="45.72" y="99.06" size="1.27" layer="95"/>
-</segment>
-<segment>
-<pinref part="IC9" gate="A" pin="G"/>
-<wire x1="40.64" y1="60.96" x2="45.72" y2="60.96" width="0.1524" layer="91"/>
-<label x="45.72" y="60.96" size="1.27" layer="95"/>
-</segment>
 </net>
 <net name="VCC" class="0">
@@
 </segment>
 </net>
-<net name="RW_OUT" class="0">
+<net name="AMIGA_ADR_ENABLE" class="0">
+<segment>
+<pinref part="IC4" gate="A" pin="G"/>
+<wire x1="40.64" y1="139.7" x2="45.72" y2="139.7" width="0.1524" layer="91"/>
+<label x="45.72" y="139.7" size="1.27" layer="95"/>
+</segment>
+<segment>
+<pinref part="IC8" gate="A" pin="G"/>
+<wire x1="40.64" y1="99.06" x2="45.72" y2="99.06" width="0.1524" layer="91"/>
+<label x="45.72" y="99.06" size="1.27" layer="95"/>
+</segment>
+<segment>
+<pinref part="IC9" gate="A" pin="G"/>
+<wire x1="40.64" y1="60.96" x2="45.72" y2="60.96" width="0.1524" layer="91"/>
+<label x="45.72" y="60.96" size="1.27" layer="95"/>
+</segment>
+</net>
+<net name="R/W" class="0">
 <segment>
 <pinref part="IC9" gate="A" pin="A1"/>

Commit message: New PCB and start for RW-Signal-Optimization
Parts:
- removed R3, R9: 4,7k, rcl:R-EU_R0603
- added RN4, RN5, RN6, RN7, RN8, RN9: 4,7k, resistor-dil:4R-NEXBV8V
Connections:
- removed net RAM_SEL: IC7.CLK1/I1, R2.1, X1-A16.B
- net A0: now also RN9A.1; no longer R3.1
- net A1: now also RN9B.1
- net A10: now also RN7C.1
- net A11: now also RN7D.1
- net A12: now also RN6A.1
- net A13: now also RN6B.1
- net A14: now also RN6C.1
- net A15: now also RN6D.1
- net A16: now also RN5A.1
- net A17: now also RN5B.1
- net A18: now also RN5C.1
- net A19: now also RN5D.1
- net A2: now also RN9C.1
- net A20: now also RN4A.1
- net A21: now also RN4B.1
- net A22: now also RN4C.1
- net A23: now also RN4D.1
- net A3: now also RN9D.1
- net A4: now also RN8A.1
- net A5: now also RN8B.1
- net A6: now also RN8C.1
- net A7: now also RN8D.1
- net A8: now also RN7A.1
- net A9: now also RN7B.1
- net GND: now also RN4A.2, RN4B.2, RN4C.2, RN4D.2, RN5A.2, RN5B.2, RN5C.2, RN5D.2, RN6A.2, RN6B.2, RN6C.2, RN6D.2, RN7A.2, RN7B.2, RN7C.2, RN7D.2, RN8A.2, RN8B.2, RN8C.2, RN8D.2, RN9A.2, RN9B.2, RN9C.2, RN9D.2; no longer R3.2
- net IO_EXP: now also IC7.CLK1/I1, R2.1, X1-A16.B; no longer R9.2
- net VCC: no longer R9.1
Other:
- moved on the sheet: C16, C17, C24, C25, C26, C27, C28, IC10P, IC11P, IC4P, IC5P, IC6P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
