File: Layout and PCB/68030-TK-V09d.brd (EAGLE design)
At the start: 92.9 x 100.2 mm, 73 parts, among them IC10 74HCT245DW, IC11 74HCT245DW, IC4 74HCT245DW, IC5 74HCT245DW, IC6 74HCT245DW, IC8 74HCT245DW, IC9 74HCT245DW, X1 FABC96R

Commit message: Cache-Disable-Option on PCB
Parts:
- added R24: 4,7k, rcl:R0603
- moved R12 2.13 mm to (64.2, 52.9)
- moved R21 2.13 mm to (64.2, 55.0)
Connections:
- net CDIS: now also R24.1
- net GND: now also R24.2
Routing:
- net GND: track 140.6 -> 146.1 mm, vias 169 -> 168
- net CDIS: track 9.09 -> 13.4 mm
- net VCC: track 151.0 -> 152.0 mm
- net MMUDIS: track 3.54 -> 4.43 mm
Changed lines of the file:
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@@
 <attribute name="NAME" x="75.1586" y="54.3814" size="0.8128" layer="25" rot="R180"/>
 </element>
-<element name="R12" library="rcl" package="R0603" value="4,7k" x="64.1604" y="50.7492" smashed="yes">
-<attribute name="NAME" x="63.2206" y="49.2506" size="0.8128" layer="25"/>
+<element name="R12" library="rcl" package="R0603" value="4,7k" x="64.1604" y="52.8828" smashed="yes">
+<attribute name="NAME" x="65.8114" y="52.6034" size="0.8128" layer="25"/>
 </element>
 <element name="R13" library="rcl" package="R0603" value="4,7k" x="79.0956" y="33.0708" smashed="yes" rot="R90">
@@
 <attribute name="NAME" x="78.7146" y="26.8986" size="0.8128" layer="25" rot="R270"/>
 </element>
-<element name="R21" library="rcl" package="R0603" value="4,7k" x="64.1604" y="52.8828" smashed="yes">
-<attribute name="NAME" x="65.8114" y="52.2986" size="0.8128" layer="25"/>
+<element name="R21" library="rcl" package="R0603" value="4,7k" x="64.1604" y="55.0164" smashed="yes">
+<attribute name="NAME" x="65.8114" y="54.4322" size="0.8128" layer="25"/>
 </element>
 <element name="RN2" library="resistor-dil" package="EXBV8V" value="4,7k" x="79.248" y="71.628" smashed="yes" rot="R90">
@@
 <attribute name="NAME" x="72.8218" y="50.0126" size="0.8128" layer="25"/>
 </element>
+<element name="R24" library="rcl" package="R0603" value="4,7k" x="64.1604" y="50.7492" smashed="yes">
+<attribute name="NAME" x="63.373" y="49.2506" size="0.8128" layer="25"/>
+</element>
 </elements>
 <signals>
@@
 <contactref element="IC1" pad="F13"/>
 <contactref element="R21" pad="1"/>
-<wire x1="59.7662" y1="52.8828" x2="63.3104" y2="52.8828" width="0.1524" layer="1"/>
+<wire x1="59.7662" y1="52.8828" x2="60.5028" y2="52.8828" width="0.1524" layer="1"/>
+<wire x1="60.5028" y1="52.8828" x2="62.6364" y2="55.0164" width="0.1524" layer="1"/>
+<wire x1="62.6364" y1="55.0164" x2="63.3104" y2="55.0164" width="0.1524" layer="1"/>
 </signal>
 <signal name="CDIS">
 <contactref element="IC1" pad="H12"/>
 <contactref element="R12" pad="1"/>
-<wire x1="61.2648" y1="48.006" x2="61.2648" y2="49.8348" width="0.1524" layer="1"/>
-<wire x1="61.2648" y1="49.8348" x2="62.1792" y2="50.7492" width="0.1524" layer="1"/>
-<wire x1="62.1792" y1="50.7492" x2="63.3104" y2="50.7492" width="0.1524" layer="1"/>
+<wire x1="61.2648" y1="48.006" x2="61.2648" y2="51.9684" width="0.1524" layer="1"/>
+<wire x1="61.2648" y1="51.9684" x2="62.1792" y2="52.8828" width="0.1524" layer="1"/>
+<wire x1="62.1792" y1="52.8828" x2="63.3104" y2="52.8828" width="0.1524" layer="1"/>
 <wire x1="57.2262" y1="47.8028" x2="58.0898" y2="46.9392" width="0.1524" layer="1"/>
 <wire x1="58.0898" y1="46.9392" x2="60.198" y2="46.9392" width="0.1524" layer="1"/>
 <wire x1="60.198" y1="46.9392" x2="61.2648" y2="48.006" width="0.1524" layer="1"/>
+<contactref element="R24" pad="1"/>
+<wire x1="63.3104" y1="50.7492" x2="63.3104" y2="52.8828" width="0.1524" layer="1"/>
 </signal>
 <signal name="STATUS">
@@
 <contactref element="R18" pad="1"/>
 <contactref element="R19" pad="1"/>
-<wire x1="65.0104" y1="50.7492" x2="65.0104" y2="52.8828" width="0.1524" layer="1"/>
+<wire x1="65.0104" y1="52.8828" x2="65.0104" y2="55.0164" width="0.1524" layer="1"/>
 <wire x1="42.5082" y1="56.8706" x2="41.9862" y2="57.3926" width="0.6096" layer="1"/>
 <wire x1="41.9862" y1="57.3926" x2="41.9862" y2="60.5028" width="0.6096" layer="1"/>
@@
 <wire x1="5.4864" y1="1.7894" x2="5.3734" y2="1.6764" width="0.8128" layer="1"/>
 <wire x1="10.9728" y1="37.214" x2="10.9728" y2="38.862" width="0.8128" layer="1"/>
-<wire x1="65.0104" y1="52.8828" x2="65.0104" y2="54.4712" width="0.1524" layer="1"/>
-<wire x1="65.0104" y1="54.4712" x2="64.4652" y2="55.0164" width="0.1524" layer="1"/>
-<via x="64.4652" y="55.0164" extent="1-16" drill="0.3"/>
+<wire x1="65.0104" y1="55.0164" x2="65.0104" y2="54.4712" width="0.1524" layer="1"/>
+<via x="65.0748" y="57.7596" extent="1-16" drill="0.3"/>
 <wire x1="75.3872" y1="44.6532" x2="75.3986" y2="44.6646" width="0.4064" layer="1"/>
 <wire x1="75.3986" y1="44.6646" x2="75.3986" y2="46.609" width="0.4064" layer="1"/>
@@
 <wire x1="72.9116" y1="49.0728" x2="72.2376" y2="49.7468" width="0.1524" layer="1"/>
 <wire x1="72.2376" y1="49.7468" x2="72.2376" y2="52.578" width="0.1524" layer="1"/>
+<wire x1="65.0748" y1="57.7596" x2="65.0748" y2="55.0808" width="0.1524" layer="1"/>
+<wire x1="65.0748" y1="55.0808" x2="65.0104" y2="55.0164" width="0.1524" layer="1"/>
 </signal>
 <signal name="GND">
@@
 <via x="62.992" y="58.0136" extent="1-16" drill="0.3"/>
 <via x="69.7484" y="58.42" extent="1-16" drill="0.3"/>
-<via x="62.8396" y="55.372" extent="1-16" drill="0.3"/>
-<via x="65.4304" y="55.3212" extent="1-16" drill="0.3"/>
 <via x="60.7568" y="86.5124" extent="1-16" drill="0.3"/>
 <via x="46.5328" y="84.4804" extent="1-16" drill="0.3"/>
@@
 <wire x1="15.24" y1="42.037" x2="16.764" y2="42.037" width="0.1524" layer="1"/>
 <wire x1="16.764" y1="42.037" x2="16.7894" y2="42.0624" width="0.1524" layer="1"/>
+<contactref element="R24" pad="2"/>
+<wire x1="65.0104" y1="50.7492" x2="65.0104" y2="48.0704" width="0.1524" layer="1"/>
+<wire x1="65.0104" y1="48.0704" x2="66.1416" y2="46.9392" width="0.1524" layer="1"/>
+<wire x1="66.1416" y1="46.9392" x2="66.1416" y2="45.72" width="0.1524" layer="1"/>
+<via x="66.1416" y="45.72" extent="1-16" drill="0.3"/>
 </signal>
 <signal name="A27">
