File: Layout and PCB/68030-TK-V09d.brd (EAGLE design)
At the start: 92.9 x 100.2 mm, 74 parts, among them IC10 74HCT245DW, IC11 74HCT245DW, IC4 74HCT245DW, IC5 74HCT245DW, IC6 74HCT245DW, IC8 74HCT245DW, IC9 74HCT245DW, X1 FABC96R

Commit message: Reset-Problem solved
The AMiga was not able to recover from a reste, because the e-clock was
not generated properly during reste.
Parts:
- R10, R11, R14: value (none) -> 68
- R16: value (none) -> 10
Changed lines of the file:
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@@
 <?xml version="1.0" encoding="utf-8"?>
 <!DOCTYPE eagle SYSTEM "eagle.dtd">
-<eagle version="6.4">
+<eagle version="6.6.0">
 <drawing>
 <settings>
@@
 <attribute name="NAME" x="7.8868" y="68.6204" size="0.8128" layer="25"/>
 </element>
-<element name="R10" library="rcl" package="R0603" value="" x="31.496" y="78.8162" smashed="yes" rot="R270">
+<element name="R10" library="rcl" package="R0603" value="68" x="31.496" y="78.8162" smashed="yes" rot="R270">
 <attribute name="NAME" x="29.3878" y="79.2988" size="0.8128" layer="25" rot="R270"/>
 <attribute name="VALUE" x="29.591" y="79.4512" size="1.27" layer="27" rot="R270"/>
 </element>
-<element name="R11" library="rcl" package="R0603" value="" x="30.6832" y="81.8134" smashed="yes" rot="R270">
+<element name="R11" library="rcl" package="R0603" value="68" x="30.6832" y="81.8134" smashed="yes" rot="R270">
 <attribute name="NAME" x="28.7274" y="82.9056" size="0.8128" layer="25" rot="R270"/>
 <attribute name="VALUE" x="28.7782" y="82.4484" size="1.27" layer="27" rot="R270"/>
 </element>
-<element name="R14" library="rcl" package="R0603" value="" x="58.674" y="85.6488" smashed="yes" rot="R180">
+<element name="R14" library="rcl" package="R0603" value="68" x="58.674" y="85.6488" smashed="yes" rot="R180">
 <attribute name="NAME" x="59.309" y="85.0138" size="0.8128" layer="25" rot="R180"/>
 <attribute name="VALUE" x="59.309" y="87.5538" size="1.27" layer="27" rot="R180"/>
 </element>
-<element name="R16" library="rcl" package="R0603" value="" x="25.4508" y="89.3064" smashed="yes" rot="R90">
+<element name="R16" library="rcl" package="R0603" value="10" x="25.4508" y="89.3064" smashed="yes" rot="R90">
 <attribute name="NAME" x="27.559" y="88.9762" size="1.27" layer="25" rot="R90"/>
 <attribute name="VALUE" x="27.3558" y="88.6714" size="1.27" layer="27" rot="R90"/>
