File: Layout and PCB/68030-TK-V09e.brd (EAGLE design)
At the start: 92.9 x 100.2 mm, 75 parts, among them IC10 74HCT245DW, IC11 74HCT245DW, IC4 74HCT245DW, IC5 74HCT245DW, IC6 74HCT245DW, IC8 74HCT245DW, IC9 74HCT245DW, X1 FABC96R

Commit message: Reset-Problem solved
The AMiga was not able to recover from a reste, because the e-clock was
not generated properly during reste.
Parts:
- added R26, R27: 4,7K, rcl:R0603
Connections:
- new net N$3: IC9.18, R26.1
- new net N$4: IC9.2, R27.2
- net GND: no longer IC9.2
- net VCC: now also R26.2, R27.1
Routing:
- net N$3: track 0.00 -> 9.72 mm
- net N$4: track 0.00 -> 5.36 mm
- net VCC: track 154.6 -> 159.0 mm, vias 34 -> 35
- net GND: track 146.1 -> 144.5 mm, vias 168 -> 167
