File: Layout and PCB/68030-TK-V09g.brd (EAGLE design)
At the start: 92.9 x 100.2 mm, 79 parts, among them IC10 74HCT245DW, IC11 74HCT245DW, IC12 100Mhz, IC4 74HCT245DW, IC5 74HCT245DW, IC6 74HCT245DW, IC8 74HCT245DW, IC9 74HCT245DW, X1 FABC96R

Commit message: Resetfix in PCB
Parts:
- moved RN1 2.59 mm to (76.7, 68.1)
- moved RN2 2.59 mm to (76.7, 71.6)
- moved RN3 2.59 mm to (76.7, 75.1)
- moved RN4 2.59 mm to (76.7, 78.6)
- moved RN5 2.59 mm to (76.7, 82.1)
- moved RN6 2.59 mm to (76.7, 85.6)
- moved RN7 2.59 mm to (76.7, 89.2)
- moved RN8 2.13 mm to (82.8, 97.1)
Routing:
- net A9: track 102.0 -> 104.6 mm
- net A8: track 104.3 -> 106.9 mm
- net A7: track 98.9 -> 101.5 mm
- net A6: track 119.1 -> 121.7 mm
- net A4: track 198.3 -> 200.9 mm
- net A31: track 89.5 -> 92.1 mm
- net A30: track 82.9 -> 85.5 mm
- net A3: track 194.2 -> 196.8 mm
- net A29: track 92.4 -> 95.0 mm
- net A28: track 92.6 -> 95.2 mm
- net A27: track 86.8 -> 89.4 mm
- net A26: track 96.9 -> 99.5 mm
- net A25: track 91.5 -> 94.1 mm
- net A24: track 84.5 -> 87.1 mm
- net A23: track 116.6 -> 119.2 mm
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Other:
- board text added: "a1k.org 68030-TK v0.9g (c) 2014 Matthias Heinrichs thx BukoCharly, Georg Braun, Herzi"
- board text removed: "a1k.org 68030-TK v0.9d (c) 2014 Matthias Heinrichs thx BukoCharly, Georg Braun, Herzi"
